Commit message: Imported upstream version '100.0.0' of 'upstream'

File: realsense2_description/urdf/_d415.urdf.xacro (robot description, xacro)
@@ -48,5 +48,4 @@
             <mesh filename="package://realsense2_description/meshes/d415.stl" />
           </geometry>
-          <material name="aluminum"/>
         </xacro:if>
         <xacro:unless value="${use_mesh}">
